Commit message: gui added

File: install/kinova_description/share/kinova_description/urdf/j2n6s300.xacro (robot description, xacro)
@@ -51,5 +51,5 @@
     <xacro:property name="joint_1_upper_limit" value="${2*J_PI}" />
     <xacro:property name="joint_1_velocity_limit" value="${36*J_PI/180}" />
-    <xacro:property name="joint_1_torque_limit" value="40" />
+    <xacro:property name="joint_1_torque_limit" value="80" />
     <xacro:property name="joint_2" value="joint_2" />
     <xacro:property name="joint_2_type" value="revolute" />
@@ -69,5 +69,5 @@
     <xacro:property name="joint_3_upper_limit" value="${341/180*J_PI}" />
     <xacro:property name="joint_3_velocity_limit" value="${36*J_PI/180}" />
-    <xacro:property name="joint_3_torque_limit" value="40" />
+    <xacro:property name="joint_3_torque_limit" value="80" />
     <xacro:property name="joint_4" value="joint_4" />
     <xacro:property name="joint_4_type" value="continuous" />
