Commit message: mejoras gui

File: src/kinova_description/urdf/j2n6s300_standalone.xacro (robot description, xacro)
@@ -1,20 +1,18 @@
 <?xml version="1.0"?>
-<!-- j2n6s300 refers to jaco v2 6DOF non-spherical 3fingers -->
 <robot xmlns:xi="http://www.w3.org/2001/XInclude"
-	xmlns:gazebo="http://playerstage.sourceforge.net/gazebo/xmlschema/#gz"
-    xmlns:model="http://playerstage.sourceforge.net/gazebo/xmlschema/#model"
-	xmlns:sensor="http://playerstage.sourceforge.net/gazebo/xmlschema/#sensor"
-	xmlns:body="http://playerstage.sourceforge.net/gazebo/xmlschema/#body"
-    xmlns:geom="http://playerstage.sourceforge.net/gazebo/xmlschema/#geom"
-    xmlns:joint="http://playerstage.sourceforge.net/gazebo/xmlschema/#joint"
-	xmlns:controller="http://playerstage.sourceforge.net/gazebo/xmlschema/#controller"
-	xmlns:interface="http://playerstage.sourceforge.net/gazebo/xmlschema/#interface"
-	xmlns:rendering="http://playerstage.sourceforge.net/gazebo/xmlschema/#rendering"
-    xmlns:renderable="http://playerstage.sourceforge.net/gazebo/xmlschema/#renderable"
-    xmlns:physics="http://playerstage.sourceforge.net/gazebo/xmlschema/#physics"
-	xmlns:xacro="http://www.ros.org/wiki/xacro" name="j2n6s300">
+  xmlns:gazebo="http://playerstage.sourceforge.net/gazebo/xmlschema/#gz"
+  xmlns:model="http://playerstage.sourceforge.net/gazebo/xmlschema/#model"
+  xmlns:sensor="http://playerstage.sourceforge.net/gazebo/xmlschema/#sensor"
+  xmlns:body="http://playerstage.sourceforge.net/gazebo/xmlschema/#body"
+  xmlns:geom="http://playerstage.sourceforge.net/gazebo/xmlschema/#geom"
+  xmlns:joint="http://playerstage.sourceforge.net/gazebo/xmlschema/#joint"
+  xmlns:controller="http://playerstage.sourceforge.net/gazebo/xmlschema/#controller"
+  xmlns:interface="http://playerstage.sourceforge.net/gazebo/xmlschema/#interface"
+  xmlns:rendering="http://playerstage.sourceforge.net/gazebo/xmlschema/#rendering"
+  xmlns:renderable="http://playerstage.sourceforge.net/gazebo/xmlschema/#renderable"
+  xmlns:physics="http://playerstage.sourceforge.net/gazebo/xmlschema/#physics"
+  xmlns:xacro="http://www.ros.org/wiki/xacro" name="j2n6s300">
   <xacro:include filename="$(find kinova_description)/urdf/j2n6s300.xacro"/>
   <link name="root"/>
-  <!-- for gazebo -->
   <link name="world"/>
   <joint name="connect_root_and_world" type="fixed">
@@ -80,15 +78,21 @@
     </plugin>
   </gazebo>
-<gazebo reference="j2n6s300_joint_finger_tip_1">
+  <gazebo reference="j2n6s300_joint_finger_tip_1">
     <implicitSpringDamper>true</implicitSpringDamper>
-    <dynamics damping="5.0" friction="10.0"/>
+    <springStiffness>50.0</springStiffness>
+    <springReference>0.0</springReference>
+    <dynamics damping="0.8" friction="0.1"/>
   </gazebo>
   <gazebo reference="j2n6s300_joint_finger_tip_2">
     <implicitSpringDamper>true</implicitSpringDamper>
-    <dynamics damping="5.0" friction="10.0"/>
+    <springStiffness>50.0</springStiffness>
+    <springReference>0.0</springReference>
+    <dynamics damping="0.8" friction="0.1"/>
   </gazebo>
   <gazebo reference="j2n6s300_joint_finger_tip_3">
     <implicitSpringDamper>true</implicitSpringDamper>
-    <dynamics damping="5.0" friction="10.0"/>
+    <springStiffness>50.0</springStiffness>
+    <springReference>0.0</springReference>
+    <dynamics damping="0.8" friction="0.1"/>
   </gazebo>
   <gazebo reference="j2n6s300_link_finger_tip_1"><mu1>2.0</mu1><mu2>2.0</mu2></gazebo>
